Commit message: Fixed .gitignore and finalized submission assets

File: so-arm/so101_ws/src/so101_description/urdf/so101_new_calib.urdf (robot description, URDF)
Before this commit: robot so101_new_calib, 8 links, 7 joints
Joints:
- joint wrist_flex: limit lower=-1.65806 upper=1.65806 effort=10 velocity=10 -> lower=-1.75 upper=1.75 effort=10 velocity=10

File: so-arm/so101_ws/src/so101_moveit_config/config/so101_new_calib.ros2_control.xacro (robot description, xacro)
@@ -33,4 +33,5 @@
                   <param name="initial_value">${initial_positions['shoulder_pan']}</param>
                 </state_interface>
+                <state_interface name="velocity"/>
                 <state_interface name="effort"/>
             </joint>
@@ -40,4 +41,5 @@
                   <param name="initial_value">${initial_positions['shoulder_lift']}</param>
                 </state_interface>
+                <state_interface name="velocity"/>
                 <state_interface name="effort"/>
             </joint>
@@ -47,4 +49,5 @@
                   <param name="initial_value">${initial_positions['elbow_flex']}</param>
                 </state_interface>
+                <state_interface name="velocity"/>
                 <state_interface name="effort"/>
             </joint>
@@ -54,4 +57,5 @@
                   <param name="initial_value">${initial_positions['wrist_flex']}</param>
                 </state_interface>
+                <state_interface name="velocity"/>
                 <state_interface name="effort"/>
             </joint>
@@ -61,4 +65,5 @@
                   <param name="initial_value">${initial_positions['wrist_roll']}</param>
                 </state_interface>
+                <state_interface name="velocity"/>
                 <state_interface name="effort"/>
             </joint>
@@ -68,4 +73,5 @@
                   <param name="initial_value">${initial_positions['gripper']}</param>
                 </state_interface>
+                <state_interface name="velocity"/>
                 <state_interface name="effort"/>
             </joint>
